File: revA.brd (EAGLE design)
At the start: 58.1 x 61 mm, 23 parts

Commit message: revA done
Parts:
- removed 3.3V: (no value), SparkFun-PowerIC:78XXL
- removed C3: (no value), SparkFun-Passives:CAP-PTH-SMALL
- removed LOGO2: OSHW-LOGOL-TOP, SparkFun-Aesthetics:OSHW_LOGO_L_TOP
- removed R10: 2.2K, SparkFun-Passives:AXIAL-0.4
- added 3V: (no value), v-reg:78LXX
- added C5: (no value), SparkFun-Passives:CAP-PTH-5MM
- added FUNC_GEN, VMEM, VOUT, VTHRESH: (no value), SparkFun-Connectors:SCREWTERMINAL-3.5MM-2
- added R0: (no value), SparkFun-Electromechanical:ALPS_POT
- 5V: device SparkFun-PowerIC:78XXL -> v-reg:78LXX
- C4: value (none) -> 0.01uF; device SparkFun-Passives:CAP-PTH-SMALL -> SparkFun-Passives:CAP-PTH-5MM
- R1, R2, R3, R4, R5: device SparkFun-Passives:AXIAL-0.4 -> SparkFun-Electromechanical:ALPS_POT
- R6: value 20K -> (none); device SparkFun-Passives:AXIAL-0.4 -> SparkFun-Electromechanical:ALPS_POT
- R7: value 10K -> (none); device SparkFun-Passives:AXIAL-0.4 -> SparkFun-Electromechanical:ALPS_POT
- R8: value 500 -> (none); device SparkFun-Resistors:AXIAL-0.4 -> SparkFun-Electromechanical:ALPS_POT
- R9: value 3.3K -> (none); device SparkFun-Passives:AXIAL-0.4 -> SparkFun-Electromechanical:ALPS_POT
- moved R9 234.7 mm to (63.5, 67.3), turned to 180 degrees
- moved R8 220.6 mm to (63.5, 54.6), turned to 180 degrees
- moved C4 211.9 mm to (50.9, 59.7), turned to 90 degrees
- moved Q 200.7 mm to (39.4, 33.0)
- moved 5V 169.8 mm to (12.7, 62.2), turned to 90 degrees
- moved R5 159.2 mm to (44.5, 6.35), turned to 90 degrees
- moved LOGO1 125.0 mm to (25.4, 19.1)
- moved PWR 117.7 mm to (5.08, 71.1), turned to 270 degrees
- moved R2 72.9 mm to (19.1, 6.35), turned to 90 degrees
- moved C2 68.2 mm to (53.3, 52.1), turned to 90 degrees
- moved R7 56.7 mm to (63.5, 41.9), turned to 180 degrees
- moved IC1 55.7 mm to (43.8, 66.0)
- moved R6 55.1 mm to (63.5, 29.2), turned to 180 degrees
- moved R4 49.3 mm to (57.1, 6.35), turned to 90 degrees
- moved C1 43.4 mm to (39.4, 26.7)
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Connections:
- removed net N$3: R10.P$1, R3.P$1, R9.P$1
- new net HAND_INPUT: R0.P$2, R2.P$1, R2.P$2
- new net R7: R6.P$2, R7.P$2, R7.P$3
- net 10V: now also 3V.IN, R0.P$1, R6.P$3, R9.P$1, U$1.P$20; no longer 3.3V.IN, R10.P$2, R5.P$2
- net 2: now also OP.6, R1.P$3, R2.P$3, R3.P$2, R3.P$3; no longer OP.2, R1.P$2, R2.P$1
- net 3.3V: now also 3V.OUT, OP.10; no longer 3.3V.OUT, OP.12
- net 5V: now also FUNC_GEN.2, OP.12, OP.5, R0.P$3, VMEM.1, VOUT.1, VTHRESH.1; no longer OP.10, OP.3
- net CON: now also C4.2; no longer C4.1
- net GND: now also 3V.GND, C4.1, C5.2, U$1.P$12, U$1.P$21; no longer 3.3V.GND, C3.2, C4.2
- net INPUT: now also FUNC_GEN.1, R1.P$2
- net N$1: now also C5.1, R9.P$2, R9.P$3; no longer C3.1, R5.P$1
- net N$2: now also R5.P$3; no longer R8.P$2
- net N$4: now also OP.9, R4.P$1, R5.P$1; no longer OP.13, R6.P$2, R7.P$1
- net N$9: now also OP.13, R7.P$1, R8.P$2, R8.P$3; no longer OP.9, R3.P$2, R4.P$1
- net TRI: now also OP.1; no longer OP.7
- net VMEM: now also OP.3, OP.7, R3.P$1, VMEM.2; no longer OP.1, OP.5, R2.P$2
- net VOUT: now also R4.P$2, R4.P$3; no longer R9.P$2
- net VOUT-: now also OP.8, R5.P$2, VOUT.2; no longer OP.14, R7.P$2, R8.P$1
- net VTHRESH: now also OP.14, OP.2, R8.P$1, VTHRESH.2; no longer OP.6, OP.8, R4.P$2
Routing:
- net 10V: track 0.00 -> 109.4 mm, vias 0 -> 3
- net VMEM: track 0.00 -> 93.9 mm, vias 0 -> 4
- net VOUT-: track 0.00 -> 77.9 mm, vias 0 -> 2
- net VOUT: track 0.00 -> 76.5 mm, vias 0 -> 3
- net INPUT: track 0.00 -> 71.8 mm, vias 0 -> 2
- net 2: track 0.00 -> 67.6 mm
- net VTHRESH: track 0.00 -> 67.0 mm
- net 5V: track 0.00 -> 53.8 mm
- net N$4: track 0.00 -> 47.8 mm
- net GND: track 0.00 -> 38.5 mm, vias 0 -> 4
- net N$9: track 0.00 -> 20.3 mm
- net N$2: track 0.00 -> 19.5 mm, vias 0 -> 2
- net HAND_INPUT: track 0.00 -> 18.2 mm
- net R7: track 0.00 -> 18.2 mm
- net TRI: track 0.00 -> 16.1 mm
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- added copper zone on layer 16, net 10V
- added copper zone on layer 16, net 5V
- added copper zone on layer 16, net GND
- added copper zone on layer 16, net N$1
- added copper zone on layer 1, net VOUT
Other:
- board size 58.1 x 61 mm -> 74.6 x 78.7 mm
- board text added: "AnalogNeuron"
- board text added: "RevA"

Commit message: fixed drc
Routing:
- net GND: track 38.5 -> 69.0 mm, vias 4 -> 8
- net VOUT-: track 77.9 -> 103.8 mm
- net VTHRESH: track 67.0 -> 91.5 mm, vias 0 -> 2
- net VMEM: track 93.9 -> 116.8 mm
- net 10V: track 109.4 -> 95.3 mm, vias 3 -> 4
- net 5V: track 53.8 -> 56.4 mm
